Commit message: re export urdf with tool joint

File: urdf/rs_m90e7_description.urdf (robot description, URDF)
Before this commit: robot robot_urdf_rs_m90e7, 6 links, 5 joints
Links:
- added link tool, mass 14.348; collision mesh filename=package://rs_m90e7_description/meshes/tool.STL; visual mesh filename=package://rs_m90e7_description/meshes/tool.STL
- link base_link: mass 14.3478185896065 -> 14.348; geometry collision mesh filename=package://rs_m90e7_description/meshes/base_link.STL; visual mesh filename=package://rs_m90e7_description/meshes/base_link.STL
- link link1: geometry collision mesh filename=package://rs_m90e7_description/meshes/link1.STL; visual mesh filename=package://rs_m90e7_description/meshes/link1.STL
- link link2: geometry collision mesh filename=package://rs_m90e7_description/meshes/link2.STL; visual mesh filename=package://rs_m90e7_description/meshes/link2.STL
- link link3: geometry collision mesh filename=package://rs_m90e7_description/meshes/link3.STL; visual mesh filename=package://rs_m90e7_description/meshes/link3.STL
- link link4: geometry collision mesh filename=package://rs_m90e7_description/meshes/link4.STL; visual mesh filename=package://rs_m90e7_description/meshes/link4.STL
- link link5: mass 14.3478185896065 -> 14.348; geometry collision mesh filename=package://rs_m90e7_description/meshes/link5.STL; visual mesh filename=package://rs_m90e7_description/meshes/link5.STL
Joints:
- added joint j6: type continuous, parent link5, child tool, origin xyz=0.08085 0.0634 0 rpy=-1.5708 1.5708 3.1416, axis 0 1 0
- joint j1: origin xyz=0 0 0.10095 rpy=1.5707963267949 0 0 -> xyz=0 0 0.10095 rpy=1.5708 0 0
- joint j2: axis 0 -1 0 -> 0 1 0; origin xyz=-0.0689499999999999 0.10315001358329 0 rpy=-3.14159265358979 0 -1.5707963267949 -> xyz=-0.06895 0.10315 0 rpy=-3.1416 0 -1.5708
- joint j3: origin xyz=-0.43 0 0 rpy=3.14159265358979 -1.5707963267949 0 -> xyz=-0.43 0 0 rpy=0 -1.5708 0
- joint j4: axis 0 -1 0 -> 0 1 0; origin xyz=-0.409999999999999 -0.0139499492415285 0 rpy=3.14159265358979 1.5707963267949 0 -> xyz=-0.41 -0.01395 0 rpy=3.1416 1.5708 0
- joint j5: axis 0 -1 0 -> 0 1 0; origin xyz=0.0678999492415284 0.0633999999999992 0 rpy=1.5707963267949 -1.5707963267949 0 -> xyz=0.0679 0.0634 0 rpy=1.5708 -1.5708 0

Commit message: 修正joint3 joint5的配置 讓0度姿態與文件一致

File: urdf/rs_m90e7_description.urdf (robot description, URDF)
Before this commit: robot rs_m90e7_description, 7 links, 6 joints
Joints:
- joint j3: origin xyz=-0.43 0 0 rpy=0 -1.5708 0 -> xyz=-0.43 0 0 rpy=3.1416 -1.5708 0
- joint j5: origin xyz=0.0679 0.0634 0 rpy=1.5708 -1.5708 0 -> xyz=0.0679 0.0634 0 rpy=-1.5708 -1.5708 0

Commit message: 修正j2 j4 j6旋轉方向與說明文件一致

File: urdf/rs_m90e7_description.urdf (robot description, URDF)
Before this commit: robot rs_m90e7_description, 7 links, 6 joints
Joints:
- joint j2: axis 0 1 0 -> 0 -1 0
- joint j4: axis 0 1 0 -> 0 -1 0
- joint j6: axis 0 1 0 -> 0 -1 0

Commit message: 更新 動作範圍(rad) 最大速度(rad/s) 容許的負荷扭矩(Nm)

File: urdf/rs_m90e7_description.urdf (robot description, URDF)
Before this commit: robot rs_m90e7_description, 7 links, 6 joints
Joints:
- joint j1: limit (none) -> lower=-6.2831853072 upper=6.2831853072 effort=0 velocity=4.7123889804; type continuous -> revolute
- joint j2: limit (none) -> lower=-6.2831853072 upper=6.2831853072 effort=0 velocity=4.7123889804; type continuous -> revolute
- joint j3: limit (none) -> lower=-4.0491638646 upper=1.2566370614 effort=0 velocity=7.1558499332; type continuous -> revolute
- joint j4: limit (none) -> lower=-6.2831853072 upper=6.2831853072 effort=16.9 velocity=8.290313947; type continuous -> revolute
- joint j5: limit (none) -> lower=-6.2831853072 upper=6.2831853072 effort=18.9 velocity=8.290313947; type continuous -> revolute
- joint j6: limit (none) -> lower=-6.2831853072 upper=6.2831853072 effort=10.2 velocity=13.1772358526; type continuous -> revolute

Commit message: stl -> dae

File: urdf/rs_m90e7_description.urdf (robot description, URDF)
Before this commit: robot rs_m90e7_description, 7 links, 6 joints
Links:
- link base_link: geometry collision mesh filename=package://rs_m90e7_description/meshes/base_link.dae; visual mesh filename=package://rs_m90e7_description/meshes/base_link.dae
- link link1: geometry collision mesh filename=package://rs_m90e7_description/meshes/link1.dae; visual mesh filename=package://rs_m90e7_description/meshes/link1.dae
- link link2: geometry collision mesh filename=package://rs_m90e7_description/meshes/link2.dae; visual mesh filename=package://rs_m90e7_description/meshes/link2.dae
- link link3: geometry collision mesh filename=package://rs_m90e7_description/meshes/link3.dae; visual mesh filename=package://rs_m90e7_description/meshes/link3.dae
- link link4: geometry collision mesh filename=package://rs_m90e7_description/meshes/link4.dae; visual mesh filename=package://rs_m90e7_description/meshes/link4.dae
- link link5: geometry collision mesh filename=package://rs_m90e7_description/meshes/link5.dae; visual mesh filename=package://rs_m90e7_description/meshes/link5.dae
- link tool: geometry collision mesh filename=package://rs_m90e7_description/meshes/tool.dae; visual mesh filename=package://rs_m90e7_description/meshes/tool.dae

Commit message: 修正j3 j4 j5模型的間隙 修正base_link的方向讓其與說明文件一至 新增tool0的座標系統並讓其姿態與說明文件dh參數的座標系統6一致 用作視覺化dae網格的品質提高 用作碰撞偵測的網格改為精簡的stl 更新readme的圖片

File: urdf/rs_m90e7_description.urdf (robot description, URDF)
Before this commit: robot rs_m90e7_description, 7 links, 6 joints
Links:
- removed link tool
- added link link6, mass 14.348; collision mesh filename=package://rs_m90e7_description/meshes/link6.stl; visual mesh filename=package://rs_m90e7_description/meshes/link6.dae
- added link tool0
- link base_link: geometry collision mesh filename=package://rs_m90e7_description/meshes/base_link.stl; visual mesh filename=package://rs_m90e7_description/meshes/base_link.dae
- link link1: mass 14.3478185896065 -> 14.348; geometry collision mesh filename=package://rs_m90e7_description/meshes/link1.stl; visual mesh filename=package://rs_m90e7_description/meshes/link1.dae
- link link2: mass 14.3478185896065 -> 14.348; geometry collision mesh filename=package://rs_m90e7_description/meshes/link2.stl; visual mesh filename=package://rs_m90e7_description/meshes/link2.dae
- link link3: mass 14.3478185896065 -> 14.348; geometry collision mesh filename=package://rs_m90e7_description/meshes/link3.stl; visual mesh filename=package://rs_m90e7_description/meshes/link3.dae
- link link4: mass 14.3478185896065 -> 14.348; geometry collision mesh filename=package://rs_m90e7_description/meshes/link4.stl; visual mesh filename=package://rs_m90e7_description/meshes/link4.dae
- link link5: geometry collision mesh filename=package://rs_m90e7_description/meshes/link5.stl; visual mesh filename=package://rs_m90e7_description/meshes/link5.dae
Joints:
- added joint jtool: type fixed, parent link6, child tool0, origin xyz=0 -0.0734 0 rpy=0 1.5708 -1.5708
- joint j1: limit lower=-6.2831853072 upper=6.2831853072 effort=0 velocity=4.7123889804 -> lower=-6.2832 upper=6.2832 effort=0 velocity=4.7124; origin xyz=0 0 0.10095 rpy=1.5708 0 0 -> xyz=0 0 0.10095 rpy=1.5708 0 1.5708
- joint j2: limit lower=-6.2831853072 upper=6.2831853072 effort=0 velocity=4.7123889804 -> lower=-6.2832 upper=6.2832 effort=0 velocity=4.7124; origin xyz=-0.06895 0.10315 0 rpy=-3.1416 0 -1.5708 -> xyz=-0.06895 0.10315 0 rpy=3.1416 0 -1.5708
- joint j3: limit lower=-4.0491638646 upper=1.2566370614 effort=0 velocity=7.1558499332 -> lower=-4.0492 upper=1.2566 effort=0 velocity=7.1558
- joint j4: limit lower=-6.2831853072 upper=6.2831853072 effort=16.9 velocity=8.290313947 -> lower=-6.2832 upper=6.2832 effort=16.9 velocity=8.2903; origin xyz=-0.41 -0.01395 0 rpy=3.1416 1.5708 0 -> xyz=-0.41 -0.0217 0 rpy=3.1416 1.5708 0
- joint j5: limit lower=-6.2831853072 upper=6.2831853072 effort=18.9 velocity=8.290313947 -> lower=-6.2832 upper=6.2832 effort=18.9 velocity=8.2903; origin xyz=0.0679 0.0634 0 rpy=-1.5708 -1.5708 0 -> xyz=0.07565 0.0634 0 rpy=-1.5708 -1.5708 0
- joint j6: axis 0 -1 0 -> 0 1 0; child tool -> link6; limit lower=-6.2831853072 upper=6.2831853072 effort=10.2 velocity=13.1772358526 -> lower=-6.2832 upper=6.2832 effort=10.2 velocity=13.177; origin xyz=0.08085 0.0634 0 rpy=-1.5708 1.5708 3.1416 -> xyz=0.08085 0.0634 0 rpy=1.5708 -1.5708 0

Commit message: 讓質量參數的執行與重量在rviz顯示正常

File: urdf/rs_m90e7_description.urdf (robot description, URDF)
Before this commit: robot rs_m90e7_description, 8 links, 7 joints
Links:
- link base_link: mass 14.348 -> 0.91957
- link link1: mass 14.348 -> 2.09505
- link link2: mass 14.348 -> 6.55317
- link link3: mass 14.348 -> 2.72253
- link link4: mass 14.348 -> 0.832958
- link link5: mass 14.348 -> 0.832958
- link link6: mass 14.348 -> 0.391580

Commit message: modify moment of inertia matrix

File: urdf/rs_m90e7_description.urdf (robot description, URDF)
Before this commit: robot rs_m90e7_description, 8 links, 7 joints
Links:
- link link1: mass 2.09505 -> 2.095055
Joints:
- removed joint j1
- removed joint j2
- removed joint j3
- removed joint j4
- removed joint j5
- removed joint j6
- added joint joint1: type revolute, parent base_link, child link1, origin xyz=0 0 0.10095 rpy=1.5708 0 1.5708, axis 0 1 0, limit lower=-6.2832 upper=6.2832 effort=0 velocity=4.7124
- added joint joint2: type revolute, parent link1, child link2, origin xyz=-0.06895 0.10315 0 rpy=3.1416 0 -1.5708, axis 0 -1 0, limit lower=-6.2832 upper=6.2832 effort=0 velocity=4.7124
- added joint joint3: type revolute, parent link2, child link3, origin xyz=-0.43 0 0 rpy=3.1416 -1.5708 0, axis 0 1 0, limit lower=-4.0492 upper=1.2566 effort=0 velocity=7.1558
- added joint joint4: type revolute, parent link3, child link4, origin xyz=-0.41 -0.0217 0 rpy=3.1416 1.5708 0, axis 0 -1 0, limit lower=-6.2832 upper=6.2832 effort=16.9 velocity=8.2903
- added joint joint5: type revolute, parent link4, child link5, origin xyz=0.07565 0.0634 0 rpy=-1.5708 -1.5708 0, axis 0 1 0, limit lower=-6.2832 upper=6.2832 effort=18.9 velocity=8.2903
- added joint joint6: type revolute, parent link5, child link6, origin xyz=0.08085 0.0634 0 rpy=1.5708 -1.5708 0, axis 0 1 0, limit lower=-6.2832 upper=6.2832 effort=10.2 velocity=13.177
