Commit message: 橋個位置

File: urdf/rs_m90e7.urdf.xacro (robot description, xacro)
@@ -13,17 +13,17 @@
     <xacro:rs_m90e7 prefix="robot1_" parent="world">
         <!-- position robot in the world -->
-        <origin xyz="1 1 0" rpy="0 0 0" />
+        <origin xyz="0.5 0.5 0" rpy="0 0 ${-135*pi/180}" />
     </xacro:rs_m90e7>
     <xacro:rs_m90e7 prefix="robot2_" parent="world">
         <!-- position robot in the world -->
-        <origin xyz="-1 1 0" rpy="0 0 0" />
+        <origin xyz="-0.5 0.5 0" rpy="0 0 ${-45*pi/180}" />
     </xacro:rs_m90e7>
     <xacro:rs_m90e7 prefix="robot3_" parent="world">
         <!-- position robot in the world -->
-        <origin xyz="-1 -1 0" rpy="0 0 0" />
+        <origin xyz="-0.5 -0.5 0" rpy="0 0 ${45*pi/180}" />
     </xacro:rs_m90e7>
     <xacro:rs_m90e7 prefix="robot4_" parent="world">
         <!-- position robot in the world -->
-        <origin xyz="1 -1 0" rpy="0 0 0" />
+        <origin xyz="0.5 -0.5 0" rpy="0 0 ${135*pi/180}" />
     </xacro:rs_m90e7>
     <!-- ========================================= -->

Commit message: URDF描述的機器人格式，統一由macro.xacro產生 update readme

File: urdf/rs_m90e7.urdf.xacro (robot description, xacro)
@@ -6,24 +6,7 @@
     <!-- ========================================= -->
     <xacro:include filename="$(find rs_m90e7_description)/urdf/rs_m90e7/rs_m90e7_macro.xacro"/>
-    <!-- ========================================= -->
-    <!-- define robot-->
-    <!-- ========================================= -->
-    <!-- create link fixed to the "world" -->
-    <link name="world" />
-    <xacro:rs_m90e7 prefix="robot1_" parent="world">
+    <xacro:rs_m90e7 prefix="" parent="">
         <!-- position robot in the world -->
-        <origin xyz="0.5 0.5 0" rpy="0 0 ${-135*pi/180}" />
-    </xacro:rs_m90e7>
-    <xacro:rs_m90e7 prefix="robot2_" parent="world">
-        <!-- position robot in the world -->
-        <origin xyz="-0.5 0.5 0" rpy="0 0 ${-45*pi/180}" />
-    </xacro:rs_m90e7>
-    <xacro:rs_m90e7 prefix="robot3_" parent="world">
-        <!-- position robot in the world -->
-        <origin xyz="-0.5 -0.5 0" rpy="0 0 ${45*pi/180}" />
-    </xacro:rs_m90e7>
-    <xacro:rs_m90e7 prefix="robot4_" parent="world">
-        <!-- position robot in the world -->
-        <origin xyz="0.5 -0.5 0" rpy="0 0 ${135*pi/180}" />
+        <origin xyz="0 0 0" rpy="0 0 0" />
     </xacro:rs_m90e7>
     <!-- ========================================= -->

File: urdf/rs_m90e7/rs_m90e7_macro.xacro (robot description, xacro)
@@ -118,5 +118,5 @@
         <inertia
           ixx=" 0.003560"
-          ixy=" -0.000889"
+          ixy="-0.000889"
           ixz=" 0.000000"
           iyy=" 0.080167"
@@ -267,10 +267,13 @@
       <child link="${prefix}flange" />
     </joint>
-    <!-- base_joint fixes base_link to the environment -->
-    <joint name="${prefix}base_joint" type="fixed">
-      <xacro:insert_block name="origin" />
-      <parent link="${parent}" />
-      <child link="${prefix}base_link" />
-    </joint>
+    <!-- 檢查${prefix}參數再決定該區快要不要輸出 -->
+    <xacro:if value="${parent != ''}">
+      <!-- base_joint fixes base_link to the environment -->
+      <joint name="${prefix}base_joint" type="fixed">
+        <xacro:insert_block name="origin" />
+        <parent link="${parent}" />
+        <child link="${prefix}base_link" />
+      </joint>
+    </xacro:if>
   </xacro:macro>
 </robot>
