Commit message: regenerate urdf

File: urdf/rs_m90e7.urdf (robot description, URDF)
Before this commit: robot rs_m90e7, 8 links, 7 joints
Links:
- link base_link: mass 0.91957 -> 1.0
- link link1: mass 2.095055 -> 5.600
- link link2: mass 6.55317 -> 13.799
- link link3: mass 2.72253 -> 4.137
- link link4: mass 0.832958 -> 2.000
- link link5: mass 0.832958 -> 2.000
- link link6: mass 0.391580 -> 0.395
Joints:
- joint joint6: axis 0 1 0 -> 0 -1 0; origin xyz=0.08085 0.0634 0 rpy=1.5708 -1.5708 0 -> xyz=0.08085 0.0634 0 rpy=-1.5708 -1.5708 0
- joint jointf: origin xyz=0 -0.0734 0 rpy=0 1.5708 -1.5708 -> xyz=0 0.0734 0 rpy=0 -1.5708 -1.5708

File: urdf/rs_m90e7/rs_m90e7_macro.xacro (robot description, xacro)
@@ -214,7 +214,4 @@
            -0.000790"
           rpy="0 0 0" />
-0.000790
-0.002215
-0.037943
         <mass
           value="0.395" />

Commit message: modify link3 origin

File: urdf/rs_m90e7.urdf (robot description, URDF)
Before this commit: robot rs_m90e7, 8 links, 7 joints
Joints:
- joint joint3: origin xyz=-0.43 0 0 rpy=3.1416 -1.5708 0 -> xyz=-0.43 0.01 0 rpy=3.1416 -1.5708 0
- joint joint4: origin xyz=-0.41 -0.0217 0 rpy=3.1416 1.5708 0 -> xyz=-0.41 -0.0117 0 rpy=3.1416 1.5708 0

File: urdf/rs_m90e7/rs_m90e7_macro.xacro (robot description, xacro)
@@ -26,5 +26,5 @@
         </geometry>
         <material name="">
-          <color rgba="0 0 0 1" />
+          <color rgba="1 1 1 1" />
         </material>
       </visual>
@@ -60,5 +60,5 @@
         </geometry>
         <material name="">
-          <color rgba="0 0 0 1" />
+          <color rgba="1 1 1 1" />
         </material>
       </visual>
@@ -94,5 +94,5 @@
         </geometry>
         <material name="">
-          <color rgba="0 0 0 1" />
+          <color rgba="1 1 1 1" />
         </material>
       </visual>
@@ -128,5 +128,5 @@
         </geometry>
         <material name="">
-          <color rgba="0 0 0 1" />
+          <color rgba="1 1 1 1" />
         </material>
       </visual>
@@ -162,5 +162,5 @@
         </geometry>
         <material name="">
-          <color rgba="0 0 0 1" />
+          <color rgba="1 1 1 1" />
         </material>
       </visual>
@@ -196,5 +196,5 @@
         </geometry>
         <material name="">
-          <color rgba="0 0 0 1" />
+          <color rgba="1 1 1 1" />
         </material>
       </visual>
@@ -230,5 +230,5 @@
         </geometry>
         <material name="">
-          <color rgba="0 0 0 1" />
+          <color rgba="1 1 1 1" />
         </material>
       </visual>
@@ -267,5 +267,5 @@
     </joint>
     <joint name="${prefix}joint3" type="revolute">
-      <origin xyz="-0.43 0 0" rpy="3.1416 -1.5708 0" />
+      <origin xyz="-0.43 0.01 0" rpy="3.1416 -1.5708 0" />
       <parent link="${prefix}link2" />
       <child link="${prefix}link3" />
@@ -274,5 +274,5 @@
     </joint>
     <joint name="${prefix}joint4" type="revolute">
-      <origin xyz="-0.41 -0.0217 0" rpy="3.1416 1.5708 0" />
+      <origin xyz="-0.41 -0.0117 0" rpy="3.1416 1.5708 0" />
       <parent link="${prefix}link3" />
       <child link="${prefix}link4" />
