Commit message: 將joint的名稱改成與ros2_control demo裡的r6bot一致

File: urdf/rs_m90e7/rs_m90e7_macro.xacro (robot description, xacro)
@@ -46,5 +46,5 @@
       </collision>
     </link>
-    <joint name="${prefix}j1" type="revolute">
+    <joint name="${prefix}joint1" type="revolute">
       <origin xyz="0 0 0.10095" rpy="1.5708 0 1.5708" />
       <parent link="${prefix}base_link" />
@@ -75,5 +75,5 @@
       </collision>
     </link>
-    <joint name="${prefix}j2" type="revolute">
+    <joint name="${prefix}joint2" type="revolute">
       <origin xyz="-0.06895 0.10315 0" rpy="3.1416 0 -1.5708" />
       <parent link="${prefix}link1" />
@@ -104,5 +104,5 @@
       </collision>
     </link>
-    <joint name="${prefix}j3" type="revolute">
+    <joint name="${prefix}joint3" type="revolute">
       <origin xyz="-0.43 0 0" rpy="3.1416 -1.5708 0" />
       <parent link="${prefix}link2" />
@@ -133,5 +133,5 @@
       </collision>
     </link>
-    <joint name="${prefix}j4" type="revolute">
+    <joint name="${prefix}joint4" type="revolute">
       <origin xyz="-0.41 -0.0217 0" rpy="3.1416 1.5708 0" />
       <parent link="${prefix}link3" />
@@ -162,5 +162,5 @@
       </collision>
     </link>
-    <joint name="${prefix}j5" type="revolute">
+    <joint name="${prefix}joint5" type="revolute">
       <origin xyz="0.07565 0.0634 0" rpy="-1.5708 -1.5708 0" />
       <parent link="${prefix}link4" />
@@ -191,5 +191,5 @@
       </collision>
     </link>
-    <joint name="${prefix}j6" type="revolute">
+    <joint name="${prefix}joint6" type="revolute">
       <origin xyz="0.08085 0.0634 0" rpy="1.5708 -1.5708 0" />
       <parent link="${prefix}link5" />

Commit message: 正名tool0為flange 將xarco的inertial參數更新

File: urdf/rs_m90e7/rs_m90e7_macro.xacro (robot description, xacro)
@@ -4,7 +4,16 @@
     <link name="${prefix}base_link">
       <inertial>
-        <origin xyz="0.10064 0.44638 0.10194" rpy="0 0 0" />
-        <mass value="14.348" />
-        <inertia ixx="0.84393" ixy="-0.35224" ixz="-0.0031091" iyy="0.54482" iyz="-0.070067" izz="1.2019" />
+        <origin
+          xyz="0.00004 0.01193 0.05418"
+          rpy="0 0 0" />
+        <mass
+          value="0.91957" />
+        <inertia
+          ixx=" 0.003109"
+          ixy="-0.000002"
+          ixz="-0.000001"
+          iyy=" 0.002643"
+          iyz="-0.000092"
+          izz=" 0.003424" />
       </inertial>
       <visual>
@@ -26,7 +35,16 @@
     <link name="${prefix}link1">
       <inertial>
-        <origin xyz="-0.10194 0.34543 0.10064" rpy="0 0 0" />
-        <mass value="14.348" />
-        <inertia ixx="1.2019" ixy="0.070067" ixz="0.0031091" iyy="0.54482" iyz="-0.35224" izz="0.84393" />
+        <origin
+          xyz="-0.009177 0.089530 0.000000"
+          rpy="0 0 0" />
+        <mass
+          value="2.095055" />
+        <inertia
+          ixx=" 0.006074"
+          ixy="-0.000305"
+          ixz=" 0.000000"
+          iyy=" 0.004584"
+          iyz=" 0.000000"
+          izz=" 0.006717" />
       </inertial>
       <visual>
@@ -55,7 +73,16 @@
     <link name="${prefix}link2">
       <inertial>
-        <origin xyz="-0.24228 0.032993 -0.10064" rpy="0 0 0" />
-        <mass value="14.348" />
-        <inertia ixx="0.54482" ixy="0.070067" ixz="-0.35224" iyy="1.2019" iyz="0.0031091" izz="0.84393" />
+        <origin
+          xyz="-0.21500 0.09444 0.00000"
+          rpy="0 0 0" />
+        <mass
+          value="6.55317" />
+        <inertia
+          ixx=" 0.015891"
+          ixy=" 0.000000"
+          ixz=" 0.000000"
+          iyy=" 0.206360"
+          iyz=" 0.000000"
+          izz=" 0.210906" />
       </inertial>
       <visual>
@@ -84,7 +111,16 @@
     <link name="${prefix}link3">
       <inertial>
-        <origin xyz="-0.10064 -0.032993 0.18772" rpy="0 0 0" />
-        <mass value="14.348" />
-        <inertia ixx="0.84393" ixy="-0.0031091" ixz="-0.35224" iyy="1.2019" iyz="-0.070067" izz="0.54482" />
+        <origin
+          xyz="-0.19905 0.05265 0.00000"
+          rpy="0 0 0" />
+        <mass
+          value="2.72253" />
+        <inertia
+          ixx=" 0.003560"
+          ixy=" -0.000889"
+          ixz=" 0.000000"
+          iyy=" 0.080167"
+          iyz=" 0.000000"
+          izz=" 0.081015" />
       </inertial>
       <visual>
@@ -113,7 +149,16 @@
     <link name="${prefix}link4">
       <inertial>
-        <origin xyz="-0.18772 0.011293 -0.30936" rpy="0 0 0" />
-        <mass value="14.348" />
-        <inertia ixx="0.54482" ixy="-0.070067" ixz="-0.35224" iyy="1.2019" iyz="-0.0031091" izz="0.84393" />
+        <origin
+          xyz="0.015396 0.057512 0.000000"
+          rpy="0 0 0" />
+        <mass
+          value="0.832958" />
+        <inertia
+          ixx=" 0.000897"
+          ixy=" 0.000092"
+          ixz=" 0.000000"
+          iyy=" 0.001490"
+          iyz=" 0.000000"
+          izz=" 0.001595" />
       </inertial>
       <visual>
@@ -142,7 +187,16 @@
     <link name="${prefix}link5">
       <inertial>
-        <origin xyz="-0.30936 -0.26337 -0.052107" rpy="0 0 0" />
-        <mass value="14.348" />
-        <inertia ixx="0.84393" ixy="-0.35224" ixz="-0.0031091" iyy="0.54482" iyz="-0.070067" izz="1.2019" />
+        <origin
+          xyz="0.015396 0.057512 0.000000"
+          rpy="0 0 0" />
+        <mass
+          value="0.832958" />
+        <inertia
+          ixx=" 0.000897"
+          ixy=" 0.000092"
+          ixz=" 0.000000"
+          iyy=" 0.001490"
+          iyz=" 0.000000"
+          izz=" 0.001595" />
       </inertial>
       <visual>
@@ -171,7 +225,16 @@
     <link name="${prefix}link6">
       <inertial>
-        <origin xyz="-0.052107 0.39021 0.32677" rpy="0 0 0" />
-        <mass value="14.348" />
-        <inertia ixx="1.2019" ixy="0.0031091" ixz="0.070067" iyy="0.84393" iyz="-0.35224" izz="0.54482" />
+        <origin
+          xyz="0.000045 -0.035542 0.000000"
+          rpy="0 0 0" />
+        <mass
+          value="0.391580" />
+        <inertia
+          ixx=" 0.000327"
+          ixy=" 0.000000"
+          ixz=" 0.000000"
+          iyy=" 0.000360"
+          iyz=" 0.000000"
+          izz=" 0.000326" />
       </inertial>
       <visual>
@@ -198,9 +261,9 @@
       <limit lower="-6.2832" upper="6.2832" effort="10.2" velocity="13.177" />
     </joint>
-    <link name="${prefix}tool0"/>
-    <joint name="${prefix}jtool" type="fixed">
+    <link name="${prefix}flange"/>
+    <joint name="${prefix}jointf" type="fixed">
       <origin xyz="0 -0.0734 0" rpy="0 1.5708 -1.5708" />
       <parent link="${prefix}link6" />
-      <child link="${prefix}tool0" />
+      <child link="${prefix}flange" />
     </joint>
     <!-- base_joint fixes base_link to the environment -->

File: urdf/rs_m90e7_description.urdf (robot description, URDF)
Before this commit: robot rs_m90e7_description, 8 links, 7 joints
Links:
- removed link tool0
- added link flange
Joints:
- removed joint jtool
- added joint jointf: type fixed, parent link6, child flange, origin xyz=0 -0.0734 0 rpy=0 1.5708 -1.5708

Commit message: update mass & inertial modify link 6 direct

File: urdf/rs_m90e7/rs_m90e7_macro.xacro (robot description, xacro)
@@ -2,18 +2,21 @@
 <robot xmlns:xacro="http://www.ros.org/wiki/xacro">
   <xacro:macro name="rs_m90e7" params="prefix parent *origin">
+    <!-- ======================================================== -->
+    <!-- robot link -->
+    <!-- ======================================================== -->
     <link name="${prefix}base_link">
       <inertial>
         <origin
-          xyz="0.00004 0.01193 0.05418"
-          rpy="0 0 0" />
-        <mass
-          value="0.91957" />
-        <inertia
-          ixx=" 0.003109"
-          ixy="-0.000002"
-          ixz="-0.000001"
-          iyy=" 0.002643"
-          iyz="-0.000092"
-          izz=" 0.003424" />
+          xyz="0.00000 0.00000 0.00000"
+          rpy="0 0 0" />
+        <mass
+          value="1.0" />
+        <inertia
+          ixx=" 0.001000"
+          ixy=" 0.000000"
+          ixz=" 0.000000"
+          iyy=" 0.001000"
+          iyz=" 0.000000"
+          izz=" 0.001000" />
       </inertial>
       <visual>
@@ -36,15 +39,18 @@
       <inertial>
         <origin
-          xyz="-0.009177 0.089530 0.000000"
-          rpy="0 0 0" />
-        <mass
-          value="2.095055" />
-        <inertia
-          ixx=" 0.006074"
-          ixy="-0.000305"
-          ixz=" 0.000000"
-          iyy=" 0.004584"
-          iyz=" 0.000000"
-          izz=" 0.006717" />
+          xyz=
+          "-0.007155
+            0.074751
+            0.000996"
+          rpy="0 0 0" />
+        <mass
+          value="5.600" />
+        <inertia
+          ixx=" 0.019807"
+          iyy=" 0.013098"
+          izz=" 0.020563"
+          ixy=" 0.000000"
+          ixz=" 0.000000"
+          iyz=" 0.000000" />
       </inertial>
       <visual>
@@ -64,4 +70,189 @@
       </collision>
     </link>
+    <link name="${prefix}link2">
+      <inertial>
+        <origin
+          xyz=
+          "-0.215018
+            0.080988
+            0.000000"
+          rpy="0 0 0" />
+        <mass
+          value="13.799" />
+        <inertia
+          ixx=" 0.041621"
+          iyy=" 0.542754"
+          izz=" 0.555726"
+          ixy=" 0.000000"
+          ixz=" 0.000000"
+          iyz=" 0.000000" />
+      </inertial>
+      <visual>
+        <origin xyz="0 0 0" rpy="0 0 0" />
+        <geometry>
+          <mesh filename="package://rs_m90e7_description/meshes/link2.dae" />
+        </geometry>
+        <material name="">
+          <color rgba="0 0 0 1" />
+        </material>
+      </visual>
+      <collision>
+        <origin xyz="0 0 0" rpy="0 0 0" />
+        <geometry>
+          <mesh filename="package://rs_m90e7_description/meshes/link2.stl" />
+        </geometry>
+      </collision>
+    </link>
+    <link name="${prefix}link3">
+      <inertial>
+        <origin
+          xyz=
+          "-0.256997
+            0.061315
+           -0.000055"
+          rpy="0 0 0" />
+        <mass
+          value="4.137" />
+        <inertia
+          ixx=" 0.007112"
+          iyy=" 0.122290"
+          izz=" 0.124242"
+          ixy=" 0.000000"
+          ixz=" 0.000000"
+          iyz=" 0.000000" />
+      </inertial>
+      <visual>
+        <origin xyz="0 0 0" rpy="0 0 0" />
+        <geometry>
+          <mesh filename="package://rs_m90e7_description/meshes/link3.dae" />
+        </geometry>
+        <material name="">
+          <color rgba="0 0 0 1" />
+        </material>
+      </visual>
+      <collision>
+        <origin xyz="0 0 0" rpy="0 0 0" />
+        <geometry>
+          <mesh filename="package://rs_m90e7_description/meshes/link3.stl" />
+        </geometry>
+      </collision>
+    </link>
+    <link name="${prefix}link4">
+      <inertial>
+        <origin
+          xyz=
+          " 0.026648
+            0.059889
+            0.000116"
+          rpy="0 0 0" />
+        <mass
+          value="2.000" />
+        <inertia
+          ixx=" 0.002061"
+          iyy=" 0.003868"
+          izz=" 0.003992"
+          ixy=" 0.000000"
+          ixz=" 0.000000"
+          iyz=" 0.000000" />
+      </inertial>
+      <visual>
+        <origin xyz="0 0 0" rpy="0 0 0" />
+        <geometry>
+          <mesh filename="package://rs_m90e7_description/meshes/link4.dae" />
+        </geometry>
+        <material name="">
+          <color rgba="0 0 0 1" />
+        </material>
+      </visual>
+      <collision>
+        <origin xyz="0 0 0" rpy="0 0 0" />
+        <geometry>
+          <mesh filename="package://rs_m90e7_description/meshes/link4.stl" />
+        </geometry>
+      </collision>
+    </link>
+    <link name="${prefix}link5">
+      <inertial>
+        <origin
+          xyz=
+          " 0.026648
+            0.053986
+            0.000116"
+          rpy="0 0 0" />
+        <mass
+          value="2.000" />
+        <inertia
+          ixx=" 0.002061"
+          iyy=" 0.003868"
+          izz=" 0.003992"
+          ixy=" 0.000000"
+          ixz=" 0.000000"
+          iyz=" 0.000000" />
+      </inertial>
+      <visual>
+        <origin xyz="0 0 0" rpy="0 0 0" />
+        <geometry>
+          <mesh filename="package://rs_m90e7_description/meshes/link5.dae" />
+        </geometry>
+        <material name="">
+          <color rgba="0 0 0 1" />
+        </material>
+      </visual>
+      <collision>
+        <origin xyz="0 0 0" rpy="0 0 0" />
+        <geometry>
+          <mesh filename="package://rs_m90e7_description/meshes/link5.stl" />
+        </geometry>
+      </collision>
+    </link>
+    <link name="${prefix}link6">
+      <inertial>
+        <origin
+          xyz=
+          "-0.002215
+            0.037943
+           -0.000790"
+          rpy="0 0 0" />
+0.000790
+0.002215
+0.037943
+        <mass
+          value="0.395" />
+        <inertia
+          ixx=" 0.000411"
+          iyy=" 0.000483"
+          izz=" 0.000429"
+          ixy=" 0.000000"
+          ixz=" 0.000000"
+          iyz=" 0.000000" />
+      </inertial>
+      <visual>
+        <origin xyz="0 0 0" rpy="0 0 0" />
+        <geometry>
+          <mesh filename="package://rs_m90e7_description/meshes/link6.dae" />
+        </geometry>
+        <material name="">
+          <color rgba="0 0 0 1" />
+        </material>
+      </visual>
+      <collision>
+        <origin xyz="0 0 0" rpy="0 0 0" />
+        <geometry>
+          <mesh filename="package://rs_m90e7_description/meshes/link6.stl" />
+        </geometry>
+      </collision>
+    </link>
+    <link name="${prefix}flange"/>
+    <!-- ======================================================== -->
+    <!-- robot joint -->
+    <!-- ======================================================== -->
+    <!-- 檢查${parent}參數再決定該區快要不要輸出該joint -->
+    <xacro:if value="${parent != ''}">
+      <joint name="${prefix}base_joint" type="fixed">
+        <xacro:insert_block name="origin" />
+        <parent link="${parent}" />
+        <child link="${prefix}base_link" />
+      </joint>
+    </xacro:if>
     <joint name="${prefix}joint1" type="revolute">
       <origin xyz="0 0 0.10095" rpy="1.5708 0 1.5708" />
@@ -71,35 +262,4 @@
       <limit lower="-6.2832" upper="6.2832" effort="0" velocity="4.7124" />
     </joint>
-    <link name="${prefix}link2">
-      <inertial>
-        <origin
-          xyz="-0.21500 0.09444 0.00000"
-          rpy="0 0 0" />
-        <mass
-          value="6.55317" />
-        <inertia
-          ixx=" 0.015891"
-          ixy=" 0.000000"
-          ixz=" 0.000000"
-          iyy=" 0.206360"
-          iyz=" 0.000000"
-          izz=" 0.210906" />
-      </inertial>
-      <visual>
-        <origin xyz="0 0 0" rpy="0 0 0" />
-        <geometry>
-          <mesh filename="package://rs_m90e7_description/meshes/link2.dae" />
-        </geometry>
-        <material name="">
-          <color rgba="0 0 0 1" />
-        </material>
-      </visual>
-      <collision>
-        <origin xyz="0 0 0" rpy="0 0 0" />
-        <geometry>
-          <mesh filename="package://rs_m90e7_description/meshes/link2.stl" />
-        </geometry>
-      </collision>
-    </link>
     <joint name="${prefix}joint2" type="revolute">
       <origin xyz="-0.06895 0.10315 0" rpy="3.1416 0 -1.5708" />
@@ -109,35 +269,4 @@
       <limit lower="-6.2832" upper="6.2832" effort="0" velocity="4.7124" />
     </joint>
-    <link name="${prefix}link3">
-      <inertial>
-        <origin
-          xyz="-0.19905 0.05265 0.00000"
-          rpy="0 0 0" />
-        <mass
-          value="2.72253" />
-        <inertia
-          ixx=" 0.003560"
-          ixy="-0.000889"
-          ixz=" 0.000000"
-          iyy=" 0.080167"
-          iyz=" 0.000000"
-          izz=" 0.081015" />
-      </inertial>
-      <visual>
-        <origin xyz="0 0 0" rpy="0 0 0" />
-        <geometry>
-          <mesh filename="package://rs_m90e7_description/meshes/link3.dae" />
-        </geometry>
-        <material name="">
-          <color rgba="0 0 0 1" />
-        </material>
-      </visual>
-      <collision>
-        <origin xyz="0 0 0" rpy="0 0 0" />
-        <geometry>
-          <mesh filename="package://rs_m90e7_description/meshes/link3.stl" />
-        </geometry>
-      </collision>
-    </link>
     <joint name="${prefix}joint3" type="revolute">
       <origin xyz="-0.43 0 0" rpy="3.1416 -1.5708 0" />
@@ -147,35 +276,4 @@
       <limit lower="-4.0492" upper="1.2566" effort="0" velocity="7.1558" />
     </joint>
-    <link name="${prefix}link4">
-      <inertial>
-        <origin
-          xyz="0.015396 0.057512 0.000000"
-          rpy="0 0 0" />
-        <mass
-          value="0.832958" />
-        <inertia
-          ixx=" 0.000897"
-          ixy=" 0.000092"
-          ixz=" 0.000000"
-          iyy=" 0.001490"
-          iyz=" 0.000000"
-          izz=" 0.001595" />
-      </inertial>
-      <visual>
-        <origin xyz="0 0 0" rpy="0 0 0" />
-        <geometry>
-          <mesh filename="package://rs_m90e7_description/meshes/link4.dae" />
-        </geometry>
-        <material name="">
-          <color rgba="0 0 0 1" />
-        </material>
-      </visual>
-      <collision>
-        <origin xyz="0 0 0" rpy="0 0 0" />
-        <geometry>
-          <mesh filename="package://rs_m90e7_description/meshes/link4.stl" />
-        </geometry>
-      </collision>
-    </link>
     <joint name="${prefix}joint4" type="revolute">
       <origin xyz="-0.41 -0.0217 0" rpy="3.1416 1.5708 0" />
@@ -185,35 +283,4 @@
       <limit lower="-6.2832" upper="6.2832" effort="16.9" velocity="8.2903" />
     </joint>
-    <link name="${prefix}link5">
-      <inertial>
-        <origin
-          xyz="0.015396 0.057512 0.000000"
-          rpy="0 0 0" />
-        <mass
-          value="0.832958" />
-        <inertia
-          ixx=" 0.000897"
-          ixy=" 0.000092"
-          ixz=" 0.000000"
-          iyy=" 0.001490"
-          iyz=" 0.000000"
-          izz=" 0.001595" />
-      </inertial>
-      <visual>
-        <origin xyz="0 0 0" rpy="0 0 0" />
-        <geometry>
-          <mesh filename="package://rs_m90e7_description/meshes/link5.dae" />
-        </geometry>
-        <material name="">
-          <color rgba="0 0 0 1" />
-        </material>
-      </visual>
-      <collision>
-        <origin xyz="0 0 0" rpy="0 0 0" />
-        <geometry>
-          <mesh filename="package://rs_m90e7_description/meshes/link5.stl" />
-        </geometry>
-      </collision>
-    </link>
     <joint name="${prefix}joint5" type="revolute">
       <origin xyz="0.07565 0.0634 0" rpy="-1.5708 -1.5708 0" />
@@ -223,57 +290,16 @@
       <limit lower="-6.2832" upper="6.2832" effort="18.9" velocity="8.2903" />
     </joint>
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